File: converter_3V3_2A/converter_3V3_2A.kicad_pcb (KiCad board)
At the start: 2 copper layers, 203 x 89.1 mm, 381 parts, among them CN1 826646-2, J1 2053380002, J2 2053380002, J3 53261-0571, P1 Header 5X2IPS1-105-01-S-D, P3 0532610471, P5 Header 5X2IPS1-105-01-S-D, P8 0532610871, Q1 MOSFET-N, Q10 MOSFET-N, Q2 MOSFET-N, Q3 MOSFET-P-SI4403CDY-T1-GE3, Q4 MOSFET-P-SI4403CDY-T1-GE3, Q5 MOSFET-P-SI4403CDY-T1-GE3, Q6 MOSFET-P-SI4403CDY-T1-GE3, Q8 MOSFET-N, Q9 MOSFET-N, SW1 0532610671, SW2 0532610671, U10 TPS5430QDDARQ1, U12 MSP430F6659IPZR, U13 REF5025AQDRQ1, U14 TPS54540QDDARQ1, U15 MAX9934TAUA+, U16 MAX9934TAUA+, U17 TLV341AIDBVR, U18 MAX9934TAUA+, U19 TLV341AIDBVR, U2 TPS54540QDDARQ1, U20 MAX9934TAUA+, U21 TLV341AIDBVR, U22 MAX9934TAUA+, U24 TLV341AIDBVR, U25 MAX9934TAUA+, U26 TLV341AIDBVR, U27 MAX9934TAUA+, U28 TCA4311ADR, U3 TPS5410QDRQ1, U4 TPS5420QDRQ1, U5 ADS1248IPW, U6 FDS6898AZ, U7 DS2777G+, U9 TPS5420QDRQ1, Y1 32MHz 10ppm, Y2 32.768kHz 12.5pF

Commit message: project finished
Parts:
- removed +L1, +L2, +L3, -L1, -L2, -L3, 3V3ANT, 3V3EPS, 3V3OBDH, 5V, CC, DC, TP1, TP2, TP6, TP7, TP9, Vpanels: TEST_POINT, FloripaSatPcbLib:TEST_POINT
- removed +X, +Y, +Z, -X, -Y, -Z: Header 4_PicoBlade, FloripaSatPcbLib:HDR4 PicoBlade
- removed 3V3_ANT, 3V3_EPS_BEACON, 3V3_MCU, 3V3_OBDH, 5V_PAYLOADS_LED, VBUS_LED: DNP, FloripaSatPcbLib:0603-LED
- removed 5V_RADIO_0, 6V_RADIO_1, VBus_TP: TEST_POINT, PCB_EPS_2:TEST_POINT
- removed 5V_RADIO_0_LED, 6V_RADIO_1_LED: DNP, PCB_EPS_2:0603-LED
- removed ? (x3): , 
- removed the C1 at (74.9, 128.7)
- removed C10, C20: 5.6nF/100V, FloripaSatPcbLib:CC0603
- removed C100, C101, C108, C109, C110, C111, C112, C113, C114, C115, C116, C119, C120, C121, C122, C124, C128, C129, C40, C41, C58, C59, C63, C71, C72, C73, C74, C75, C76, C83, C84, C85, C86, C87, C88, C89, C90, C91, C93, C94, C97, C98, C99: 0.1uF/50V, FloripaSatPcbLib:CC0603
- removed C102, C103, C104, C105, C106, C107, C13, C130, C14: 4.7uF/25V, FloripaSatPcbLib:CC0805
- removed C11, C12, C126, C127, C15, C22, C25, C27, C29, C45, C47, C53, C55, C62, C77, C78: 0.1uF/50V, FloripaSatPcbLib:CC0805
- removed C117, C118, C36, C50, C51, C79, C80, C81, C82: 22uF/25V, FloripaSatPcbLib:CC1210
- removed C123, C125, C33, C35, C60, C61, C64: 10uF/10V, FloripaSatPcbLib:CC0805_Tantalum
- removed C131, C132, C16, C17, C18, C30, C48, C7, C8: 22uF/10V, FloripaSatPcbLib:CC1206
- removed C133: 0.1uF/50V, PCB_EPS_2:CC0603
- removed C19, C9: 13pF/50V, FloripaSatPcbLib:CC0603
- removed the C2 at (71.4, 131.1)
- removed C21, C26, C32, C34, C44, C52: 0.01uF/50V, FloripaSatPcbLib:CC0805
- removed C23, C28, C46, C54: 10uF/25V, FloripaSatPcbLib:CC1206
- removed C24, C31, C49, C56: 220uF/6.3V, FloripaSatPcbLib:cc1210
- removed the C3 at (72.9, 131.1)
- removed C37, C38: 1000pF/50V, FloripaSatPcbLib:CC0603
- removed C39, C65: 0.47uF/50V, FloripaSatPcbLib:CC0603
- removed the C4 at (69.9, 131.1)
- removed the C5 at (90.5, 128.9)
- removed C57: 1nF/16V, PCB_EPS_2:CC0805
- removed the C6 at (91.1, 123.4)
- removed C66: 0.01uF/25V, FloripaSatPcbLib:CC0603
- removed C67, C69: 12pF/50V, FloripaSatPcbLib:CC0603
- removed C68, C70: 10pF/100V, FloripaSatPcbLib:CC0805
- removed CN1: 826646-2, footprints_library_legacy:HDR 1X2
- removed the D1 at (83.7, 126.8)
- removed D10: B220-13-F, FloripaSatPcbLib:DO-214AA
- removed D11, D13, D15, D4, D9: B340LA-13-F, FloripaSatPcbLib:DO-214AC
- removed D12, D14, D16, D7: DNP, footprints_library_legacy:SOD323F
- removed D17, D18, D8: DNP, FloripaSatPcbLib:SOD323F
- removed D2: FSV530AF, FloripaSatPcbLib:DO-214AC
- removed D3: CMS06(TE12L,Q,M), FloripaSatPcbLib:cms06
- removed D5, D6: 3SMAJ5919B-TP, FloripaSatPcbLib:DO-214AC
- removed FB1: 30R@100Mhz, 3A, FloripaSatPcbLib:IND0805
- removed FB3, FB4: 30R@100Mhz, 10A, FloripaSatPcbLib:IND1210
- removed FD1, FD2, FD3, FD4, FD5, FD6: Fiducial 1.3, footprints_library_legacy:Fiducial 1.3mm
- removed J_V1, J_V3, J_V4, J_V5, J_V6, R28, R32, R87: 0R, FloripaSatPcbLib:0805
- removed the L1 at (81.8, 121.5)
- removed L2: 2.2uH/9A 15mOHM, FloripaSatPcbLib:Ind_SRP6540
- removed L3: 27uH/4.3A/42.5mOHM, FloripaSatPcbLib:IND_744325xxx
- removed L4, L5: 16uH/5A/34.5mOHM, FloripaSatPcbLib:IND_744325xxx
- removed L6: 10uH/6.4A/51.8mOHM, FloripaSatPcbLib:Ind_IHLP
- removed L7, L8, L9: 22uH/6.3/25.7mOHM, FloripaSatPcbLib:IND_HC9
- removed MEC1, MEC2, MEC3, MEC4, MEC5, MEC6, MEC7, MEC8, MEC9: M3, footprints_library_legacy:M3 hole
- removed P1: Header 5X2IPS1-105-01-S-D, PCB_EPS_2:IPS1-105-01-S-D
- removed P3: 0532610471, footprints_library_legacy:PICOBLADE 4PIN RIGHT ANGLE
- removed P5: Header 5X2IPS1-105-01-S-D, FloripaSatPcbLib:IPS1-105-01-S-D
- removed P8, RTD1, RTD2: 0532610871, footprints_library_legacy:PICOBLADE 8PIN RIGHT ANGLE
- removed Q1, Q10, Q2, Q8, Q9: MOSFET-N, FloripaSatPcbLib:SOIC8_Mosfet
- removed Q3, Q4, Q5, Q6: MOSFET-P-SI4403CDY-T1-GE3, FloripaSatPcbLib:SOIC8_Mosfet
- removed the R1 at (77.8, 141.5)
- removed R10, R15, R16, R20, R21, R46, R47, R50, R51, R55, R56, R9: 0R, FloripaSatPcbLib:1206
- removed R11: 60.4k, FloripaSatPcbLib:0805
- removed R12: 19.6k, FloripaSatPcbLib:0603
- removed R13, R6: 11.5k, FloripaSatPcbLib:0805
- removed R14, R7: 140k, FloripaSatPcbLib:0603
- removed R17, R22, R52, R57: 10k, FloripaSatPcbLib:0805
- removed R18, R23, R31, R34, R37, R39, R40, R43, R53, R58, R60, R61, R8: 1k, FloripaSatPcbLib:0603
- removed R19, R24, R54: 5K9, FloripaSatPcbLib:0805
- removed the R2 at (71.6, 135.6)
- removed R25, R26: 1k, FloripaSatPcbLib:0805
- removed R27: 1.65K, FloripaSatPcbLib:0805
- removed R29, R41, R49, R68, R75, R78: 0.02R/0.5W, footprints_library_legacy:1206 - ohmite
- removed the R3 at (94.8, 132.3)
- removed R30, R48, R67, R72, R77, R79: 3k3, footprints_library_legacy:R0805
- removed R33, R42, R44: 150R, FloripaSatPcbLib:0603
- removed R35, R85: 100K 1/10W, FloripaSatPcbLib:0805
- removed R36: 4.02K, FloripaSatPcbLib:0805
- removed R38: 470R, FloripaSatPcbLib:0603
- removed the R4 at (83.7, 137.3)
- removed R45, R70: 300K, FloripaSatPcbLib:0603
- removed the R5 at (84.5, 134.1)
- removed R59: 3.24k 1/8W, FloripaSatPcbLib:0805
- removed R62: 47k, FloripaSatPcbLib:0603
- removed R64: 4K7, FloripaSatPcbLib:0603
- removed R65, R66, R83, R84: 10k, footprints_library_legacy:R0603
- removed R69, R74, R81: 93K1, FloripaSatPcbLib:0603
- removed R71, R73, R76, R82, R86: 100K, FloripaSatPcbLib:0603
- removed R80: 1k, footprints_library_legacy:R0603
- removed R88, R89, R90, R91: 0R, PCB_EPS_2:0805
- removed R92: 150R, footprints_library_legacy:R0603
- removed R93: 0R, PCB_EPS_2:1206
- removed RBF: 0533980471, footprints_library_legacy:PICOBLADE 4PIN VERTICAL
- removed RSense1: 0.01R/0.5W, FloripaSatPcbLib:1206 - ohmite
- removed R_ESD: 1.2M, PCB_EPS_2:0805
- removed Rsense3: 0.075R/0.5W, FloripaSatPcbLib:1206 - ohmite
- removed SBW, SW1, SW2: 0532610671, footprints_library_legacy:PICOBLADE 6PIN Right Angle
- removed SYSTEM_FAULT: 150060RS75000, footprints_library_legacy:0603-RED-LED
- removed SYSTEM_ON: RED, FloripaSatPcbLib:0603-LED
- removed U10: TPS5430QDDARQ1, FloripaSatPcbLib:SO8 Power PAD
- removed U12: MSP430F6659IPZR, FloripaSatPcbLib:PZ0100A_N
- removed U13: REF5025AQDRQ1, FloripaSatPcbLib:SOIC-8
- removed U14: TPS54540QDDARQ1, PCB_EPS_2:SO8 Power PAD
- removed U15, U16, U18, U20, U22, U25, U27: MAX9934TAUA+, FloripaSatPcbLib:MSOP-8
- removed U17, U19, U21, U24, U26: TLV341AIDBVR, FloripaSatPcbLib:SOT-23 6L
- removed U2: TPS54540QDDARQ1, FloripaSatPcbLib:SO8 Power PAD
- removed U28: TCA4311ADR, PCB_EPS_2:SOIC8
- removed U3: TPS5410QDRQ1, FloripaSatPcbLib:SO8 Power PAD
- removed U4, U9: TPS5420QDRQ1, FloripaSatPcbLib:SO8 Power PAD
- removed U5: ADS1248IPW, FloripaSatPcbLib:TSSOP28
- removed U6: FDS6898AZ, FloripaSatPcbLib:SOIC8
- removed U7: DS2777G+, FloripaSatPcbLib:TDFN-14-EP_3x5
- removed UART: DNP, footprints_library_legacy:HDR 1X3
- removed V1, V2, V3, V4: 47k, footprints_library_legacy:0805
- removed Y1: 32MHz 10ppm, FloripaSatPcbLib:XTAL_ABM8X
- removed Y2: 32.768kHz 12.5pF, FloripaSatPcbLib:ABS06 0805
- R4, R5: value 500m -> 1R
- moved J3 28.2 mm to (151.1, 80.7)
- moved J1 28.2 mm to (110.5, 95.8)
- moved R1 28.2 mm to (126.5, 107.3)
- moved R2 28.2 mm to (127.0, 81.8)
- moved R4 28.2 mm to (119.5, 94.8)
- moved C1 28.2 mm to (127.0, 99.0)
- moved U1 28.2 mm to (128.0, 90.8)
- moved C2 28.2 mm to (127.0, 103.3)
- moved C3 28.2 mm to (136.1, 86.9)
- moved C4 28.2 mm to (166.6, 97.9)
- moved C5 28.2 mm to (161.6, 97.9)
- moved C6 28.2 mm to (156.1, 97.9)
- moved J2 28.2 mm to (184.3, 96.0)
- moved R3 28.2 mm to (131.6, 81.8)
- moved R5 28.2 mm to (172.1, 99.3)
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Routing:
- net VBus: track 116.9 -> 0.00 mm, vias 10 -> 0
- net VPANELS: track 61.5 -> 0.00 mm, vias 2 -> 0
- net MPPT_PWM_3: track 47.7 -> 0.00 mm, vias 2 -> 0
- net 3V3_DEPLOYMENT_ANT: track 43.2 -> 0.00 mm
- net -RBF: track 38.3 -> 0.00 mm, vias 4 -> 0
- net GNDREF: track 0.00 -> 35.8 mm, vias 0 -> 9
- net MPPT_PWM_2: track 35.5 -> 0.00 mm, vias 2 -> 0
- net Net+L1_1: track 34.5 -> 0.00 mm, vias 3 -> 0
- net MPPT_PWM_1: track 31.3 -> 0.00 mm, vias 2 -> 0
- net Net-L1_1: track 30.2 -> 0.00 mm, vias 2 -> 0
- net Net+L3_1: track 27.1 -> 0.00 mm, vias 2 -> 0
- net PANEL-Z: track 26.7 -> 0.00 mm, vias 2 -> 0
- net Net+L2_1: track 19.1 -> 0.00 mm, vias 3 -> 0
- net NetC55_1: track 19.0 -> 0.00 mm, vias 3 -> 0
- net +RBF: track 18.2 -> 0.00 mm, vias 4 -> 0
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- removed copper zone on F.Cu, net 6V_Radio_1
- removed copper zone on F.Cu, net Net3V3ANT_1
- removed copper zone on F.Cu, net Net3V3OBDH_1
- removed copper zone on F.Cu, net NetC11_2
- removed copper zone on F.Cu, net NetC15_1
- removed copper zone on F.Cu, net NetC1_2
- removed copper zone on F.Cu, net NetC21_2
- removed copper zone on F.Cu, net NetC26_2
- removed copper zone on F.Cu, net NetC44_2
- removed copper zone on F.Cu, net NetC47_2
- removed copper zone on F.Cu, net NetC52_2
- removed copper zone on F.Cu, net NetC55_1
- removed copper zone on F.Cu, net NetC5_1
- removed copper zone on F.Cu, net PGND
- removed copper zone on F.Cu, net VPANELS
Other:
- board size 203 x 89.1 mm -> 88.5 x 41 mm
- board text removed: "+"
- board text removed: "-"
- board text removed: "16"
- board text removed: "24"
- board text removed: "32"
- board text removed: "40"
- board text removed: "46"
- board text removed: "5V_OBDH"
- board text removed: "5V_PAYLOAD"
- board text removed: "5V_RADIO_0"
- board text removed: "6V_RADIO_1"
- board text removed: "8"
- board text removed: "ADD_GPIO"
- board text removed: "ADD_I2C"
- board text removed: "AGND"
- board text removed: "ANT_VCC"
- board text removed: "BATTERY"
- board text removed: "BAT_VCC"
- board text removed: "CHARGER"
- board text removed: "CK"
- board text removed: "DGND"
- board text removed: "DO"
- board text removed: "EN_RADIOS"
- board text removed: "EPS_I2C"
- board text removed: "GND"
- board text removed: "GPIO"
- board text removed: "H1+"
- board text removed: "H1-"
- board text removed: "H2-"
- board text removed: "HEATER"
- board text removed: "JTAG"
- board text removed: "NC1"
- board text removed: "NC2"
- board text removed: "PGND"
- board text removed: "RBF+"
- board text removed: "RBF-"
- board text removed: "RTD"
- board text removed: "RTD0"
- board text removed: "RTD1"
- board text removed: "RTD2"
- board text removed: "RTD3"
- board text removed: "RTD4"
- board text removed: "RTD5"
- board text removed: "RTD6"
- board text removed: "RX"
- board text removed: "TP1"
- board text removed: "TP2"
- board text removed: "TP9"
- board text removed: "TX"
- board text removed: "UART_RADIO_1"
- board text removed: "V+"
- board text removed: "V-"
- board text removed: "VBAT+"
- board text removed: "VBAT-"
- board text removed: "VBus_TP"
- board text removed: "VCC"
- board text removed: "V_CM"
