File: converter_3V3_2A/converter_3V3_2A.kicad_pcb (KiCad board)
At the start: 2 copper layers, 88.5 x 41 mm, 17 parts, among them J1 2053380002, J2 2053380002, J3 53261-0571

Commit message: update
Routing:
- net Net-(D1-K): track 1.90 -> 11.4 mm
Changed lines of the file:
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@@
+	)
+	(segment
+		(start 141.45 88.35)
+		(end 145.7 92.6)
+		(width 0.381)
+		(layer "B.Cu")
+		(net 4)
+	)
+	(segment
+		(start 137.95 88.35)
+		(end 141.45 88.35)
+		(width 0.381)
+		(layer "B.Cu")
+		(net 4)
 	)
 	(segment
@@
 		(start 118.55 94.85)
 		(end 114.275 94.85)
-		(width 0.25)
+		(width 0.762)
 		(layer "F.Cu")
 		(net 11)
@@
 		(start 175.05 99.35)
 		(end 179.445 94.955)
-		(width 0.25)
+		(width 0.762)
 		(layer "F.Cu")
 		(net 14)
@@
 		(start 173.05 99.35)
 		(end 175.05 99.35)
-		(width 0.25)
+		(width 0.762)
 		(layer "F.Cu")
 		(net 14)
@@
 		(start 179.445 94.955)
 		(end 180.575 94.955)
-		(width 0.25)
+		(width 0.762)
 		(layer "F.Cu")
 		(net 14)
@@
 		(start 120.55 94.85)
 		(end 120.55 102.35)
-		(width 0.25)
+		(width 0.762)
 		(layer "F.Cu")
 		(net 16)
@@
 		(start 120.55 102.35)
 		(end 125.55 107.35)
-		(width 0.25)
-		(layer "F.Cu")
-		(net 16)
+		(width 0.762)
+		(layer "F.Cu")
+		(net 16)

Commit message: needs review
Routing:
- net Net-(C4-Pad1): track 36.2 -> 62.9 mm
Changed lines of the file:
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@@
-	)
-	(segment
-		(start 124.8 95.55)
-		(end 124.8 94.85625)
-		(width 0.381)
-		(layer "F.Cu")
-		(net 1)
 	)
 	(segment
@@
 	)
 	(segment
-		(start 124.8 94.85625)
-		(end 126.05 93.60625)
-		(width 0.381)
-		(layer "F.Cu")
-		(net 1)
-	)
-	(segment
 		(start 128.5 106.4)
 		(end 127.55 107.35)
@@
 	)
 	(via
-		(at 124.8 95.55)
-		(size 0.6)
-		(drill 0.3)
-		(layers "F.Cu" "B.Cu")
-		(free yes)
+		(at 126.05 93.60625)
+		(size 0.6)
+		(drill 0.3)
+		(layers "F.Cu" "B.Cu")
+		(free yes)
+		(net 1)
+	)
+	(segment
+		(start 126.05 93.60625)
+		(end 128.59375 93.60625)
+		(width 0.381)
+		(layer "B.Cu")
+		(net 1)
+	)
+	(segment
+		(start 128.59375 93.60625)
+		(end 128.6 93.6)
+		(width 0.2)
+		(layer "B.Cu")
 		(net 1)
 	)
@@
 	)
 	(segment
+		(start 126.05 83.45)
+		(end 126.05 81.85)
+		(width 0.381)
+		(layer "F.Cu")
+		(net 5)
+	)
+	(segment
 		(start 151.1 86.9)
 		(end 151.1 81.45)
@@
 	)
 	(segment
-		(start 124.5 81.85)
-		(end 126.05 81.85)
-		(width 0.381)
-		(layer "F.Cu")
-		(net 5)
-	)
-	(segment
 		(start 171.8 94.1)
 		(end 166.8 89.1)
@@
 	)
 	(via
-		(at 124.5 81.85)
-		(size 0.6)
-		(drill 0.3)
-		(layers "F.Cu" "B.Cu")
-		(free yes)
-		(net 5)
-	)
+		(at 126.05 83.45)
+		(size 0.6)
+		(drill 0.3)
+		(layers "F.Cu" "B.Cu")
+		(free yes)
+		(net 5)
+	)
+	(segment
+		(start 143.1 100.5)
+		(end 145.6 100.5)
+		(width 0.381)
+		(layer "B.Cu")
+		(net 5)
+	)
+	(segment
+		(start 126.05 83.45)
+		(end 143.1 100.5)
+		(width 0.381)
+		(layer "B.Cu")
+		(net 5)
+	)
