File: converter_3V3_2A/converter_3V3_2A.kicad_sch (KiCad schematic)
At the start: 17 parts, among them J1 2053380002, J2 2053380002, J3 53261-0571

Commit message: project finished
Parts:
- R4, R5: value 500m -> 1R
Changed lines of the file:
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@@
 			)
 		)
-		(property "Value" "500m"
+		(property "Value" "1R"
 			(at 66.802 89.916 90)
 			(effects
@@
 			)
 		)
-		(property "Value" "500m"
+		(property "Value" "1R"
 			(at 229.362 89.916 90)
 			(effects
