File: load_converter_3V3/load_converter_3V3.kicad_pcb (KiCad board)
At the start: 2 copper layers, 170 x 91.9 mm, 418 parts, among them J1 2053380002, J1 2053380004, J10 532610271, J13 532610671, J17 532610671, J18 532610271, J19 N/A, J2 2053380004, J2 53261-0671, J20 N/A, J21 2053380002, J22 2053380002, J23 N/A, J24 N/A, J25 2053380002, J26 2053380002, J27 2053380002, J28 2053380002, J29 2053380002, J3 2053380002, J3 532610471, J4 2053380002, J4 2053380004, J5 532610471, J6 2053380002, J6 532610471, J7 532610471, J8 532610471, J9 532610671, Q1 SI2302DDS-T1-GE3, Q10 SI2302DDS-T1-GE3, Q11 EPC2016C, Q12 EPC2016C, Q13 SI2302DDS-T1-GE3, Q18 SI2302DDS-T1-GE3, Q19 SI2302DDS-T1-GE3, Q2 SI2302DDS-T1-GE3, Q20 SI2302DDS-T1-GE3, Q21 SI2302DDS-T1-GE3, Q22 SI2302DDS-T1-GE3, Q23 SI2302DDS-T1-GE3, Q24 SI7414DN-T1-E3, Q25 SI7414DN-T1-E3, Q28 EPC2016C, Q29 EPC2016C, Q3 EPC2016C, Q30 EPC2016C, Q31 EPC2016C, Q4 EPC2016C, Q5 SI7414DN-T1-E3, Q6 SI7414DN-T1-E3, Q7 SI2302DDS-T1-GE3, Q8 SI2302DDS-T1-GE3, Q9 SI2302DDS-T1-GE3, U1 INA199C3DCKR, U1 LMV321RIYLT, U10 INA199C3DCKR, U11 LMV321RIYLT, U12 NVTFS5116PLTAG, U13 NVTFS5116PLTAG, U14 NVTFS5116PLTAG, U15 CD4051BPWR, U16 CD4051BPWR, U17 NVTFS5116PLTAG, U18 NVTFS5116PLTAG, U19 INA199C3DCKR, U2 INA199C3DCKR, U2 LTC3833EUDC#TRPBF, U20 INA199C1DCKR, U21 INA199C3DCKR, U22 INA199C3DCKR, U23 LTC3833EUDC#TRPBF, U24 INA199C1DCKR, U26 LTC3833EUDC#TRPBF, U28 BQ24650RVAT, U29 LMV321RIYLT, U3 INA199C3DCKR, U30 LTC3833EUDC#TRPBF, U31 LTC3833EUDC#TRPBF, U32 BQ24650RVAT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

Commit message: needs to be revised
Parts:
- moved RGND1 65.5 mm to (148.9, 64.1), turned to 180 degrees
- moved R16 14.5 mm to (169.3, 91.5), turned to 90 degrees
- moved R1 12.4 mm to (150.3, 108.3), turned to 90 degrees
- moved J1 1.11 mm to (146.0, 117.6)
- moved J6 0.17 mm to (146.0, 54.4)
- turned C6 to 180 degrees
Routing:
- net Net-(U1-OUT): track 0.00 -> 56.8 mm
- net Net-(J1-Pad1): track 0.00 -> 51.8 mm
- net Net-(J2-Pad5): track 0.00 -> 51.3 mm, vias 0 -> 1
- net Net-(U1-IN+): track 0.00 -> 49.6 mm, vias 0 -> 1
- net GNDS3: track 2.05 -> 27.8 mm, vias 3 -> 7
- net GNDPWR: track 10.2 -> 34.2 mm, vias 27 -> 30
- net /3V3: track 2.17 -> 25.1 mm, vias 0 -> 5
- net Net-(Q30-Gate): track 4.16 -> 25.2 mm, vias 2 -> 3
- net Net-(Q28-Gate): track 2.82 -> 23.4 mm, vias 2 -> 3
- net Net-(Q9-G): track 0.00 -> 18.9 mm
- net Net-(Q9-D): track 3.23 -> 17.0 mm, vias 2 -> 3
- net Net-(D1-K): track 8.95 -> 13.1 mm, vias 2 -> 4
- net /3V3_VCC1: track 8.78 -> 12.9 mm
- net Net-(U2-PGOOD): track 0.00 -> 3.76 mm, vias 0 -> 2
- net /3V3_SENSE1+: track 0.00 -> 3.58 mm, vias 0 -> 2
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- removed copper zone on B.Cu, net GNDS3
