File: load_converter_3V3/load_converter_3V3.kicad_sch (KiCad schematic)
At the start: 46 parts, among them J1 2053380002, J2 53261-0671, J23 N/A, J3 2053380002, J4 2053380002, J6 2053380002, Q28 EPC2016C, Q30 EPC2016C, Q9 SI2302DDS-T1-GE3, U1 INA199C3DCKR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

Commit message: needs to be revised
Parts:
- R1, R16: value 100m -> 1R
Changed lines of the file:
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@@
 			)
 		)
-		(property "Value" "100m"
+		(property "Value" "1R"
 			(at 477.52 124.968 0)
 			(do_not_autoplace yes)
@@
 			)
 		)
-		(property "Value" "100m"
+		(property "Value" "1R"
 			(at 90.17 100.33 90)
 			(effects
