File: 3V3_load_converter/3V3_load_converter.kicad_sch (KiCad schematic)
At the start: 0 parts

Commit message: update
Parts:
- added H1, H2, H3, H4: Mounting hole (3.2 mm), footprints:MountingHole, symbol MountingHole:MountingHole
- added TP1, TP10, TP11, TP12, TP13, TP14, TP15, TP16, TP17, TP18, TP19, TP2, TP20, TP21, TP22, TP23, TP24, TP25, TP26, TP27, TP3, TP7, TP8, TP9: Test point, footprints:testpoint_smd, symbol TESTPOINT:TestPoint
Connections:
- net 3V3_A_~{EN}: now also TP20.1
- net 3V3_B_~{EN}: now also TP21.1
- new net 3V3_AntDep: TP10.1
- new net 3V3_Beacon: TP11.1
- new net 3V3_OBDH: TP12.1
- new net 5V0_A_~{EN}: TP18.1
- new net 5V0_B_~{EN}: TP19.1
- new net 5V0_Payload: TP7.1
- new net 5V0_RadioBeacon: TP8.1
- new net 5V0_RadioMain: TP9.1
- new net AntDep_EN: TP25.1
- new net BC_A_TS: TP16.1
- new net BC_A_~{EN}: TP14.1
- new net BC_B_TS: TP17.1
- new net BC_B_~{EN}: TP15.1
- new net BC_VFB: TP13.1
- new net Beacon_EN: TP26.1
- new net OBDH_EN: TP27.1
- new net Payload_EN: TP22.1
- new net RadioBeacon_EN: TP23.1
- new net RadioMain_EN: TP24.1
- new net VBUS: TP3.1
- new net VIN: TP2.1
- new net VPANELS: TP1.1
