File: 3V3_load_converter/MPPT_Battery_Charger.kicad_sch (KiCad schematic)
At the start: 78 parts, among them Q10 SI2302DDS-T1-GE3, Q13 SI2302DDS-T1-GE3, Q24 SI7414DN-T1-E3, Q25 SI7414DN-T1-E3, Q5 SI7414DN-T1-E3, Q6 SI7414DN-T1-E3, U20 INA199C1DCKR, U24 INA199C1DCKR, U28 BQ24650RVAT, U29 LMV321RIYLT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

Commit message: update
Parts:
- removed C42, C43, C56, C78, C79, C82, C83, C91: 100nF, footprints:CAP0603, symbol C0603C104K5RACTU:C0603C104K5RACTU
- removed C73, C74: 2.2uF, footprints:CAP1210, symbol C1210C225K5RACTU:C1210C225K5RACTU
- removed C75, C76, C77, C80, C81, C84, C87, C93: 1uF, footprints:CAP0805, symbol C0805C105K5RACTU:C0805C105K5RACTU
- removed C85, C86, C89, C92: 10uF, footprints:CAP1210, symbol C1210C106K5RACTU:C1210C106K5RACTU
- removed C88, C90: 4.7uF, footprints:CAP1210, symbol C1210C475K5RACTU:C1210C475K5RACTU
- removed D10, D9: PDS1040L-13, footprints:PDS1040L-13, symbol PDS1040L-13:PDS1040L-13
- removed D11, D12: BAT54, footprints:BAT54, symbol BAT54:BAT54
- removed D15, D16: PMEG3050EP,115, footprints:PMEG3050EP,115, symbol PMEG3050EP,115:PMEG3050EP,115
- removed D2, D3, D5, D6: LTST-C190GKT, footprints:LTST-C190GKT, symbol LTST-C190GKT:LTST-C190GKT
- removed JP5, JP6: N/A, footprints:Jumper, symbol JUMPER:JUMPER
- removed L3, L5: 12uH, footprints:744770112, symbol 744770112:744770112
- removed Q10, Q13: SI2302DDS-T1-GE3, footprints:SI2302DDS-T1-GE3, symbol SI2302DDS-T1-GE3:SI2302DDS-T1-GE3
- removed Q24, Q25, Q5, Q6: SI7414DN-T1-E3, footprints:SI7414DN-T1-E3, symbol SI7414DN-T1-E3:SI7414DN-T1-E3
- removed R100, R90: 270k, footprints:RES0805, symbol CRCW0805270KFKEAHP:CRCW0805270KFKEAHP
- removed R101, R89: 2R, footprints:RES2010, symbol CRCW20102R00FKEF:CRCW20102R00FKEF
- removed R103, R68: 5.23k, footprints:RES0603, symbol CRCW06035K23FKEAHP:CRCW06035K23FKEAHP
- removed R108, R67: 33m, footprints:RES2010, symbol WSL2010R0330FEA:WSL2010R0330FEA
- removed R109: 20m, footprints:RES2010, symbol WSL2010R0200FEA:WSL2010R0200FEA
- removed R110: 24k, footprints:RES0603, symbol CRCW060324K0FKEAHP:CRCW060324K0FKEAHP
- removed R111: 7.5k, footprints:RES0603, symbol CRCW06037K50FKEAHP:CRCW06037K50FKEAHP
- removed R115, R99: 30.1k, footprints:RES0603, symbol CRCW060330K1FKEAHP:CRCW060330K1FKEAHP
- removed R15, R87, R91, R93: 20k, footprints:RES0805, symbol CRCW080520K0FKEAHP:CRCW080520K0FKEAHP
- removed R58: 25m, footprints:RES2010, symbol WSL2010R0250FEA18:WSL2010R0250FEA18
- removed R59, R60: 10R, footprints:RES0603, symbol CRCW060310R0FKEAHP:CRCW060310R0FKEAHP
- removed R69, R70, R71, R94: 10k, footprints:RES0805, symbol RC0805FR-0710KL:RC0805FR-0710KL
- removed R72: 8.2k, footprints:RES0603, symbol CRCW06038K20FKEAHP:CRCW06038K20FKEAHP
- removed R85: 30k, footprints:RES0603, symbol CRCW060330K0FKEAHP:CRCW060330K0FKEAHP
- removed R88, R92: 100k, footprints:RES0603, symbol CRCW0603100KFKEAHP:CRCW0603100KFKEAHP
- removed U20, U24: INA199C1DCKR, footprints:INA199C1DCKR, symbol INA199C1DCKR:INA199C1DCKR
- removed U28, U32: BQ24650RVAT, footprints:BQ24650RVAT, symbol BQ24650RVAT:BQ24650RVAT
- removed U29, U35: LMV321RIYLT, footprints:LMV321RIYLT, symbol LMV321RIYLT:LMV321RIYLT
