File: 3V3_load_converter/3V3_Load_Converters.kicad_sch (KiCad schematic)
At the start: 40 parts, among them J23 N/A, Q28 EPC2016C, Q30 EPC2016C, Q9 SI2302DDS-T1-GE3, U21 INA199C3DCKR, U30 LTC3833EUDC#TRPBF

Commit message: update
Parts:
- added J1, J2: 2053380002, footprints:2053380002, symbol 2053380002:2053380002
- added J3: 532610871, footprints:CONN_532610001-SD_08_MOL, symbol 532610871:532610871
- added R1, R2: 5m, footprints:RES2010, symbol WSL20105L000FEA:WSL20105L000FEA
- added TP5: Test point, footprints:testpoint_smd, symbol TESTPOINT:TestPoint
Connections:
- net 3V3: now also J3.7, R2.1, TP5.1
- net GNDPWR: now also J1.2, J2.2, J3.6
- net at R74.1, U30.17 (PGOOD): now also J3.5
- net 3V3_A_~{EN}: no longer names the net of Q9.1 (G), R123.2
- net 3V3_A_~{EN}: now also J3.4
- net AMUX7: no longer names the net of U21.6 (OUT)
- net AMUX7: now also J3.3
- net VBUS: no longer names the net of C40.2, R29.1, U21.3 (V+), U21.4 (IN+)
- net VBUS: now also J3.2, R1.2
- new net: J1.1, J3.1, R1.1
- new net: J2.1, J3.8, R2.2
Other:
- note added: "ANALOG SIGNALS"
- note added: "POWER FLAGS"
- note added: "TEST POINTS"
- moved on the sheet: C100, C102, C104, C106, C108, C110, C112, C114, C116, C118, C120, C122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

Commit message: needs review
Connections:
- net 3V3: now also J3.6; no longer J3.7
- net GNDPWR: now also J3.8; no longer J3.6
- net at J2.1, R2.2: now also J3.7; no longer J3.8
Changed lines of the file:
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@@
 	(wire
 		(pts
-			(xy 336.55 157.48) (xy 336.55 158.75)
+			(xy 213.36 63.5) (xy 392.43 63.5)
 		)
 		(stroke
@@
 	(wire
 		(pts
-			(xy 336.55 158.75) (xy 360.68 158.75)
+			(xy 336.55 157.48) (xy 336.55 158.75)
 		)
 		(stroke
@@
 	(wire
 		(pts
-			(xy 182.88 143.51) (xy 182.88 147.32)
+			(xy 336.55 158.75) (xy 360.68 158.75)
 		)
 		(stroke
@@
 	(wire
 		(pts
-			(xy 245.11 99.06) (xy 245.11 104.14)
+			(xy 182.88 143.51) (xy 182.88 147.32)
 		)
 		(stroke
@@
 	(wire
 		(pts
-			(xy 275.59 111.76) (xy 278.13 111.76)
+			(xy 245.11 99.06) (xy 245.11 104.14)
 		)
 		(stroke
-			(width 0.5)
+			(width 0)
 			(type default)
 		)
@@
 	(wire
 		(pts
-			(xy 215.9 63.5) (xy 392.43 63.5)
+			(xy 275.59 111.76) (xy 278.13 111.76)
 		)
 		(stroke
-			(width 0)
+			(width 0.5)
 			(type default)
 		)
@@
 	(wire
 		(pts
-			(xy 213.36 66.04) (xy 383.54 66.04)
+			(xy 215.9 55.88) (xy 215.9 58.42)
 		)
 		(stroke
@@
 	(wire
 		(pts
+			(xy 210.82 66.04) (xy 210.82 55.88)
+		)
+		(stroke
+			(width 0)
+			(type default)
+		)
+	)
+	(wire
+		(pts
 			(xy 208.28 167.64) (xy 190.5 167.64)
 		)
@@
 	(wire
 		(pts
+			(xy 210.82 66.04) (xy 383.54 66.04)
+		)
+		(stroke
+			(width 0)
+			(type default)
+		)
+	)
+	(wire
+		(pts
 			(xy 347.98 120.65) (xy 347.98 135.89)
 		)
@@
 	(wire
 		(pts
-			(xy 210.82 55.88) (xy 210.82 69.85)
+			(xy 215.9 58.42) (xy 220.98 58.42)
 		)
 		(stroke
@@
 	(wire
 		(pts
+			(xy 213.36 63.5) (xy 213.36 55.88)
+		)
+		(stroke
+			(width 0)
+			(type default)
+		)
+	)
+	(wire
+		(pts
 			(xy 345.44 85.09) (xy 345.44 86.36)
 		)
@@
 	(wire
 		(pts
-			(xy 213.36 55.88) (xy 213.36 66.04)
-		)
-		(stroke
-			(width 0)
-			(type default)
-		)
-	)
-	(wire
-		(pts
-			(xy 215.9 55.88) (xy 215.9 63.5)
-		)
-		(stroke
-			(width 0)
-			(type default)
-		)
-	)
-	(wire
-		(pts
 			(xy 360.68 111.76) (xy 369.57 111.76)
 		)
@@
 	(symbol
 		(lib_id "power:GNDPWR")
-		(at 210.82 69.85 0)
+		(at 220.98 58.42 0)
 		(unit 1)
 		(exclude_from_sim no)
@@
 		(fields_autoplaced yes)
 		(property "Reference" "#PWR03"
-			(at 210.82 74.93 0)
+			(at 220.98 63.5 0)
 			(effects
 				(font
@@
 		)
 		(property "Value" "GNDPWR"
-			(at 210.693 73.66 0)
+			(at 220.853 62.23 0)
 			(effects
 				(font
@@
 		)
 		(property "Footprint" ""
-			(at 210.82 71.12 0)
+			(at 220.98 59.69 0)
 			(effects
 				(font
@@
 		)
 		(property "Datasheet" ""
-			(at 210.82 71.12 0)
+			(at 220.98 59.69 0)
 			(effects
 				(font
@@
 		)
 		(property "Description" "Power symbol creates a global label with name \"GNDPWR\" , global ground"
-			(at 210.82 69.85 0)
+			(at 220.98 58.42 0)
 			(effects
 				(font
@@
 		)
 		(instances
-			(project "eps-re_project"
+			(project "3V3_load_converter"
 				(path "/2eebaa11-d7ed-4bfd-bc8e-988f68654d29/6f34948c-43a8-4614-b8ed-90c5b6b9b243"
 					(reference "#PWR03")
