File: 3V3_load_converter/3V3_load_converter.kicad_pcb (KiCad board)
At the start: 6 copper layers, 55.8 x 49.9 mm, 40 parts, among them J23 N/A, Q28 EPC2016C, Q30 EPC2016C, Q9 SI2302DDS-T1-GE3, U21 INA199C3DCKR, U30 LTC3833EUDC#TRPBF

Commit message: update
Parts:
- removed the C100 at (81.6, 55.4)
- removed the C102 at (81.6, 56.9)
- removed the C104 at (77.6, 53.1)
- removed the C106 at (73.8, 62.1)
- removed the C108 at (78.0, 66.3)
- removed the C110 at (86.5, 67.5)
- removed the C112 at (65.4, 70.6)
- removed the C114 at (67.4, 78.1)
- removed the C116 at (67.4, 74.8)
- removed the C118 at (68.0, 80.8)
- removed the C120 at (70.0, 55.9)
- removed the C122 at (91.7, 80.4)
- removed the C124 at (84.9, 80.4)
- removed the C126 at (88.3, 80.4)
- removed the C40 at (68.3, 88.3)
- removed the C98 at (82.3, 66.0)
- removed the D13 at (90.9, 68.7)
- removed the J23 at (85.7, 58.2)
- removed the JP4 at (86.2, 74.8)
- removed the L4 at (76.9, 73.8)
- removed the Q28 at (74.5, 81.3)
- removed the Q30 at (79.9, 81.3)
- removed the Q9 at (92.1, 59.6)
- removed the R123 at (98.1, 58.6)
- removed the R127 at (78.8, 57.5)
- removed the R140 at (76.4, 57.5)
- removed the R142 at (74.8, 57.5)
- removed the R29 at (71.6, 83.7)
- removed the R64 at (71.5, 62.8)
- removed the R65 at (71.5, 61.3)
- removed the R66 at (75.4, 65.7)
- removed the R74 at (98.1, 61.5)
- removed the R78 at (86.2, 73.5)
- removed the R80 at (72.4, 55.1)
- removed the R81 at (72.4, 56.7)
- removed the R96 at (83.1, 63.6)
- removed the R97 at (82.2, 59.3)
- removed the RGND4 at (75.9, 50.3)
- removed the U21 at (68.3, 85.3)
- removed the U30 at (78.3, 62.2)
- added C100: 3.3nF, footprints:CAP0603, B.Cu at (103.9, 53.8)
- added C100: 3.3nF, footprints:CAP0603, B.Cu at (256.0, 59.2)
- added C102: 100pF, footprints:CAP0603, B.Cu at (103.9, 55.4)
- added C102: 100pF, footprints:CAP0603, B.Cu at (256.0, 60.7)
- added C104: 1nF, footprints:CAP0603, B.Cu at (99.9, 51.6)
- added C104: 1nF, footprints:CAP0603, B.Cu at (252.0, 56.9)
- added C106: 1nF, footprints:CAP0603, B.Cu at (248.2, 65.9)
- added C106: 1nF, footprints:CAP0603, B.Cu at (96.1, 60.5)
- added C108: 100nF, footprints:CAP0603, B.Cu at (252.4, 70.1)
- added C108: 100nF, footprints:CAP0603, B.Cu at (100.3, 64.7)
- added C110: 4.7uF, footprints:CAP1210, B.Cu at (260.9, 71.4)
- added C110: 4.7uF, footprints:CAP1210, B.Cu at (108.8, 66.0)
- added C112: 47uF, footprints:CAP2917POL, B.Cu at (239.8, 74.4)
- added C112: 47uF, footprints:CAP2917POL, B.Cu at (87.6, 69.1)
- added C114: 10uF, footprints:CAP1210, B.Cu at (89.7, 76.6)
- added C114: 10uF, footprints:CAP1210, B.Cu at (241.8, 81.9)
- added C116: 10uF, footprints:CAP1210, B.Cu at (89.7, 73.2)
- added C116: 10uF, footprints:CAP1210, B.Cu at (241.8, 78.6)
- added C118: 1uF, footprints:CAP0805, B.Cu at (90.3, 79.3)
- added C118: 1uF, footprints:CAP0805, B.Cu at (242.4, 84.6)
- added C120: 22pF, footprints:CAP0603, B.Cu at (244.4, 59.7)
- added C120: 22pF, footprints:CAP0603, B.Cu at (92.3, 54.4)
- added C122: 22uF, footprints:CAP1210, B.Cu at (266.0, 84.2)
- added C122: 22uF, footprints:CAP1210, B.Cu at (113.9, 78.9)
- added C124: 22uF, footprints:CAP1210, B.Cu at (259.3, 84.2)
- added C124: 22uF, footprints:CAP1210, B.Cu at (107.2, 78.9)
- added C126: 22uF, footprints:CAP1210, B.Cu at (110.6, 78.9)
- added C126: 22uF, footprints:CAP1210, B.Cu at (262.7, 84.2)
- added C40: 100nF, footprints:CAP0603, B.Cu at (242.7, 92.1)
- added C40: 100nF, footprints:CAP0603, B.Cu at (90.5, 86.8)
- added C98: 100nF, footprints:CAP0603, B.Cu at (104.5, 64.5)
- added C98: 100nF, footprints:CAP0603, B.Cu at (256.6, 69.8)
- added D13: SS12FP, footprints:SS12FP, B.Cu at (113.2, 67.2)
- added D13: SS12FP, footprints:SS12FP, B.Cu at (265.3, 72.5)
- added G***: LOGO, footprints:SpaceLab_logo, F.Cu at (101.6, 67.0)
- added G***: LOGO, footprints:open_hardware_logo, F.Cu at (102.9, 73.8)
- added G***: LOGO, footprints:qr_code_git, F.Cu at (91.4, 91.7)
- added H1: Mounting hole (3.2 mm), footprints:MountingHole, F.Cu at (44.5, 32.4)
- added H2: Mounting hole (3.2 mm), footprints:MountingHole, F.Cu at (118.2, 32.4)
- added H3: Mounting hole (3.2 mm), footprints:MountingHole, F.Cu at (40.8, 118.1)
- added H4: Mounting hole (3.2 mm), footprints:MountingHole, F.Cu at (120.8, 118.1)
- added J1: 2053380002, footprints:2053380002, F.Cu at (251.1, 105.2)
- added J2: 2053380002, footprints:2053380002, F.Cu at (264.2, 105.4)
- added J22: 2053380002, footprints:2053380002, F.Cu at (75.8, 34.3)
- added J23: N/A, footprints:three_position_jumper, B.Cu at (108.0, 56.7)
- added J23: N/A, footprints:three_position_jumper, B.Cu at (260.1, 62.0)
- added J25: 2053380002, footprints:2053380002, F.Cu at (64.6, 34.3)
- added J26: 2053380002, footprints:2053380002, F.Cu at (53.5, 34.3)
- added J27: 2053380002, footprints:2053380002, F.Cu at (107.8, 34.3)
- added J28: 2053380002, footprints:2053380002, F.Cu at (97.7, 34.3)
- added J29: 2053380002, footprints:2053380002, F.Cu at (86.7, 34.3)
- added J3: 532610871, footprints:CONN_532610001-SD_08_MOL, F.Cu at (285.5, 77.5)
- added JP4: N/A, footprints:Jumper, B.Cu at (260.6, 78.6)
- added JP4: N/A, footprints:Jumper, B.Cu at (108.5, 73.2)
- added L4: 2.4uH, footprints:744325240, B.Cu at (251.2, 77.6)
- added L4: 2.4uH, footprints:744325240, B.Cu at (99.1, 72.3)
- added Q28: EPC2016C, footprints:EPC2016C, B.Cu at (96.8, 79.8)
- added Q28: EPC2016C, footprints:EPC2016C, B.Cu at (248.9, 85.1)
- added Q30: EPC2016C, footprints:EPC2016C, B.Cu at (102.1, 79.8)
- added Q30: EPC2016C, footprints:EPC2016C, B.Cu at (254.2, 85.1)
- added Q9: SI2302DDS-T1-GE3, footprints:SI2302DDS-T1-GE3, B.Cu at (266.5, 63.4)
- added Q9: SI2302DDS-T1-GE3, footprints:SI2302DDS-T1-GE3, B.Cu at (114.4, 58.0)
- added R1: 5m, footprints:RES2010, F.Cu at (250.1, 94.1)
- added R123: 100k, footprints:RES0603, B.Cu at (272.5, 62.4)
- added R123: 100k, footprints:RES0603, B.Cu at (120.4, 57.1)
- added R127: 12k, footprints:RES0603, B.Cu at (253.2, 61.3)
- added R127: 12k, footprints:RES0603, B.Cu at (101.1, 56.0)
- added R140: 90.9k, footprints:RES0603, B.Cu at (250.8, 61.3)
- added R140: 90.9k, footprints:RES0603, B.Cu at (98.7, 56.0)
- added R142: 20k, footprints:RES0603, B.Cu at (97.1, 56.0)
- added R142: 20k, footprints:RES0603, B.Cu at (249.2, 61.3)
- added R2: 5m, footprints:RES2010, F.Cu at (263.2, 94.1)
- added R29: 5m, footprints:RES2010, B.Cu at (246.0, 87.5)
- added R29: 5m, footprints:RES2010, B.Cu at (93.8, 82.2)
- added R64: 10R, footprints:RES0603, B.Cu at (245.9, 66.6)
- added R64: 10R, footprints:RES0603, B.Cu at (93.8, 61.3)
- added R65: 10R, footprints:RES0603, B.Cu at (245.9, 65.1)
- added R65: 10R, footprints:RES0603, B.Cu at (93.8, 59.8)
- added R66: 10R, footprints:RES0603, B.Cu at (249.8, 69.5)
- added R66: 10R, footprints:RES0603, B.Cu at (97.7, 64.2)
- added R74: 100k, footprints:RES0603, B.Cu at (120.4, 60.0)
- added R74: 100k, footprints:RES0603, B.Cu at (272.5, 65.3)
- added R78: 16m, footprints:RES2010, B.Cu at (260.6, 77.3)
- added R78: 16m, footprints:RES2010, B.Cu at (108.5, 72.0)
- added R80: 0R, footprints:RES0603, B.Cu at (94.7, 53.6)
- added R80: 0R, footprints:RES0603, B.Cu at (246.8, 58.9)
- added R81: 0R, footprints:RES0603, B.Cu at (246.8, 60.5)
- added R81: 0R, footprints:RES0603, B.Cu at (94.7, 55.1)
- added R96: 2.2R, footprints:RES0603, B.Cu at (257.5, 67.4)
- added R96: 2.2R, footprints:RES0603, B.Cu at (105.4, 62.1)
- added R97: 82k, footprints:RES0603, B.Cu at (256.6, 63.1)
- added R97: 82k, footprints:RES0603, B.Cu at (104.5, 57.8)
- added RGND4: 0R, footprints:RES0603, B.Cu at (250.3, 54.1)
- added RGND4: 0R, footprints:RES0603, B.Cu at (98.2, 48.8)
- added TP4: Test point, footprints:testpoint_smd, F.Cu at (102.0, 48.9)
- added TP5: Test point, footprints:testpoint_smd, F.Cu at (102.0, 43.3)
- added U21: INA199C3DCKR, footprints:INA199C3DCKR, B.Cu at (90.5, 83.8)
- added U21: INA199C3DCKR, footprints:INA199C3DCKR, B.Cu at (242.7, 89.1)
- added U30: LTC3833EUDC#TRPBF, footprints:LTC3833EUDC#TRPBF, B.Cu at (100.6, 60.6)
- added U30: LTC3833EUDC#TRPBF, footprints:LTC3833EUDC#TRPBF, B.Cu at (252.7, 66.0)
Routing:
- net (no net): track 0.00 -> 2584.9 mm, vias 0 -> 210
- net /BC_VFB: track 0.00 -> 141.6 mm, vias 0 -> 4
- net /U_3V3_Load_Converters/3V3_VCC1: track 15.3 -> 95.8 mm, vias 4 -> 8
- net /BC_B_TS: track 0.00 -> 77.9 mm, vias 0 -> 3
- net /BC_A_~{EN}: track 0.00 -> 74.3 mm, vias 0 -> 3
- net /BC_A_TS: track 0.00 -> 68.5 mm, vias 0 -> 3
- net Net-(U30-PGOOD): track 2.71 -> 71.1 mm, vias 2 -> 5
- net /BC_B_~{EN}: track 0.00 -> 65.7 mm, vias 0 -> 2
- net /VIN: track 0.00 -> 65.3 mm, vias 0 -> 3
- net Net-(U21-OUT): track 0.00 -> 64.1 mm, vias 0 -> 4
- net +5V: track 0.00 -> 63.9 mm, vias 0 -> 22
- net /5V0_A_~{EN}: track 0.00 -> 59.9 mm, vias 0 -> 3
- net /5V0_B_~{EN}: track 0.00 -> 54.9 mm, vias 0 -> 2
- net /U_3V3_Load_Converters/3V3: track 0.00 -> 52.3 mm, vias 0 -> 20
- net /U_3V3_Load_Converters/3V3_SENSE1-: track 1.73 -> 53.8 mm, vias 2 -> 4
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- added copper zone on B.Cu, net (none)
- added copper zone on F.Cu, net (none)
- added copper zone on In2.Cu, net (none)
- added copper zone on In4.Cu, net (none)
- added copper zone on B.Cu, net +5V
- added copper zone on In3.Cu, net +5V
- added copper zone on B.Cu, net /3V3_AntDep
- added copper zone on F.Cu, net /3V3_AntDep
- added copper zone on In3.Cu, net /3V3_AntDep
- added copper zone on B.Cu, net /3V3_Beacon
- added copper zone on F.Cu, net /3V3_Beacon
- added copper zone on In3.Cu, net /3V3_Beacon
- added copper zone on B.Cu, net /3V3_OBDH
- added copper zone on F.Cu, net /3V3_OBDH
- added copper zone on In3.Cu, net /3V3_OBDH
- added copper zone on B.Cu, net /5V0_Payload
- added copper zone on F.Cu, net /5V0_Payload
- added copper zone on In3.Cu, net /5V0_Payload
- added copper zone on B.Cu, net /5V0_RadioBeacon
- added copper zone on F.Cu, net /5V0_RadioBeacon
- added copper zone on In3.Cu, net /5V0_RadioBeacon
- added copper zone on B.Cu, net /5V0_RadioMain
- added copper zone on F.Cu, net /5V0_RadioMain
- added copper zone on In3.Cu, net /5V0_RadioMain
- added copper zone on B.Cu, net /U_3V3_Load_Converters/3V3
- added copper zone on In3.Cu, net /U_3V3_Load_Converters/3V3
- added copper zone on In2.Cu, net /U_3V3_Load_Converters/VBUS_BK3V3
- added copper zone on F.Cu, net /VIN
- added copper zone on F.Cu, net /VPANELS
- added copper zone on In3.Cu, net /VPANELS
- added copper zone on B.Cu, net GNDPWR
- added copper zone on F.Cu, net GNDPWR
- added copper zone on In1.Cu, net GNDPWR
- added copper zone on In4.Cu, net GNDPWR
- added copper zone on In4.Cu, net GNDS3
- added copper zone on B.Cu, net Net-(U21-IN+)
- added copper zone on F.Cu, net Net-(U21-IN+)
- added copper zone on In2.Cu, net Net-(U21-IN+)
- removed copper zone on B.Cu, net +3V3
- removed copper zone on B.Cu, net VBUS
Other:
- board size 55.8 x 49.9 mm -> 251.3 x 91.9 mm
- board text added: "1"
- board text added: "2"
- board text added: "3"
- board text added: "4"
- board text added: "5"
- board text added: "6"
- board text added: "Layer numbering"

Commit message: needs review
Parts:
- removed the C100 at (103.9, 53.8)
- removed the C102 at (103.9, 55.4)
- removed the C104 at (99.9, 51.6)
- removed the C106 at (96.1, 60.5)
- removed the C108 at (100.3, 64.7)
- removed the C110 at (108.8, 66.0)
- removed the C112 at (87.6, 69.1)
- removed the C114 at (89.7, 76.6)
- removed the C116 at (89.7, 73.2)
- removed the C118 at (90.3, 79.3)
- removed the C120 at (92.3, 54.4)
- removed the C122 at (113.9, 78.9)
- removed the C124 at (107.2, 78.9)
- removed the C126 at (110.6, 78.9)
- removed the C40 at (90.5, 86.8)
- removed the C98 at (104.5, 64.5)
- removed the D13 at (113.2, 67.2)
- removed G***: LOGO, footprints:SpaceLab_logo
- removed G***: LOGO, footprints:open_hardware_logo
- removed G***: LOGO, footprints:qr_code_git
- removed H1, H2, H3, H4: Mounting hole (3.2 mm), footprints:MountingHole
- removed J1, J2, J22, J25, J26, J27, J28, J29: 2053380002, footprints:2053380002
- removed the J23 at (108.0, 56.7)
- removed J3: 532610871, footprints:CONN_532610001-SD_08_MOL
- removed the JP4 at (108.5, 73.2)
- removed the L4 at (99.1, 72.3)
- removed the Q28 at (96.8, 79.8)
- removed the Q30 at (102.1, 79.8)
- removed the Q9 at (114.4, 58.0)
- removed R1, R2: 5m, footprints:RES2010
- removed the R123 at (120.4, 57.1)
- removed the R127 at (101.1, 56.0)
- removed the R140 at (98.7, 56.0)
- removed the R142 at (97.1, 56.0)
- removed the R29 at (93.8, 82.2)
- removed the R64 at (93.8, 61.3)
- removed the R65 at (93.8, 59.8)
- removed the R66 at (97.7, 64.2)
- removed the R74 at (120.4, 60.0)
- removed the R78 at (108.5, 72.0)
- removed the R80 at (94.7, 53.6)
- removed the R81 at (94.7, 55.1)
- removed the R96 at (105.4, 62.1)
- removed the R97 at (104.5, 57.8)
- removed the RGND4 at (98.2, 48.8)
- removed TP4, TP5: Test point, footprints:testpoint_smd
- removed the U21 at (90.5, 83.8)
- removed the U30 at (100.6, 60.6)
- moved C108 177.0 mm to (75.5, 73.8)
- moved C110 177.0 mm to (84.0, 75.1)
- moved C114 177.0 mm to (64.9, 85.7)
- moved C116 177.0 mm to (64.9, 82.3)
- moved C118 177.0 mm to (65.5, 88.4)
- moved C122 177.0 mm to (89.1, 88.0)
- moved C126 177.0 mm to (85.8, 88.0)
- moved J23 177.0 mm to (83.2, 65.8)
- moved JP4 177.0 mm to (83.7, 82.3)
- moved L4 177.0 mm to (74.3, 81.4)
- moved Q28 177.0 mm to (72.0, 88.9)
- moved R127 177.0 mm to (76.3, 65.1)
- moved R140 177.0 mm to (73.9, 65.1)
- moved R29 177.0 mm to (69.0, 91.3)
- moved R64 177.0 mm to (69.0, 70.4)
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Routing:
- net (no net): track 2584.9 -> 0.00 mm, vias 210 -> 0
- net /BC_VFB: track 141.6 -> 0.00 mm, vias 4 -> 0
- net /BC_B_TS: track 77.9 -> 0.00 mm, vias 3 -> 0
- net /BC_A_~{EN}: track 74.3 -> 0.00 mm, vias 3 -> 0
- net /BC_A_TS: track 68.5 -> 0.00 mm, vias 3 -> 0
- net /BC_B_~{EN}: track 65.7 -> 0.00 mm, vias 2 -> 0
- net /VIN: track 65.3 -> 0.00 mm, vias 3 -> 0
- net +5V: track 63.9 -> 0.00 mm, vias 22 -> 0
- net Net-(U21-OUT): track 64.1 -> 1.59 mm, vias 4 -> 1
- net /5V0_A_~{EN}: track 59.9 -> 0.00 mm, vias 3 -> 0
- net /5V0_B_~{EN}: track 54.9 -> 0.00 mm, vias 2 -> 0
- net /U_3V3_Load_Converters/3V3: track 52.3 -> 0.00 mm, vias 20 -> 0
- net Net-(U21-IN+): track 51.8 -> 0.00 mm, vias 12 -> 0
- net +3V3: track 57.4 -> 6.31 mm, vias 20 -> 6
- net Net-(J1-Pad1): track 50.7 -> 0.00 mm, vias 3 -> 0
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- added copper zone on In3.Cu, net +3V3
- added copper zone on B.Cu, net VBUS
- added copper zone on In2.Cu, net VBUS
- removed copper zone on B.Cu, net (none)
- removed copper zone on F.Cu, net (none)
- removed copper zone on In2.Cu, net (none)
- removed copper zone on In4.Cu, net (none)
- removed copper zone on B.Cu, net +5V
- removed copper zone on In3.Cu, net +5V
- removed copper zone on B.Cu, net /3V3_AntDep
- removed copper zone on F.Cu, net /3V3_AntDep
- removed copper zone on In3.Cu, net /3V3_AntDep
- removed copper zone on B.Cu, net /3V3_Beacon
- removed copper zone on F.Cu, net /3V3_Beacon
- removed copper zone on In3.Cu, net /3V3_Beacon
- removed copper zone on B.Cu, net /3V3_OBDH
- removed copper zone on F.Cu, net /3V3_OBDH
- removed copper zone on In3.Cu, net /3V3_OBDH
- removed copper zone on B.Cu, net /5V0_Payload
- removed copper zone on F.Cu, net /5V0_Payload
- removed copper zone on In3.Cu, net /5V0_Payload
- removed copper zone on B.Cu, net /5V0_RadioBeacon
- removed copper zone on F.Cu, net /5V0_RadioBeacon
- removed copper zone on In3.Cu, net /5V0_RadioBeacon
- removed copper zone on B.Cu, net /5V0_RadioMain
- removed copper zone on F.Cu, net /5V0_RadioMain
- removed copper zone on In3.Cu, net /5V0_RadioMain
- removed copper zone on In3.Cu, net /U_3V3_Load_Converters/3V3
- removed copper zone on F.Cu, net /VIN
- removed copper zone on F.Cu, net /VPANELS
- removed copper zone on In3.Cu, net /VPANELS
- removed copper zone on F.Cu, net GNDPWR
- removed copper zone on In1.Cu, net GNDPWR
- removed copper zone on In4.Cu, net GNDPWR
- removed copper zone on B.Cu, net Net-(U21-IN+)
- removed copper zone on F.Cu, net Net-(U21-IN+)
- removed copper zone on In2.Cu, net Net-(U21-IN+)
Other:
- board size 251.3 x 91.9 mm -> 45.8 x 46.7 mm
- board text removed: "1"
- board text removed: "2"
- board text removed: "3"
- board text removed: "4"
- board text removed: "5"
- board text removed: "6"
- board text removed: "Layer numbering"
