File: 3V3_eps2_converter/3V3_eps2_converter.kicad_sch (KiCad schematic)
At the start: 15 parts

Commit message: update
Parts:
- removed FD1, FD2, FD3, FD4, FD5, FD6: Fiducial 1.3, Fiducial 1.3mm, symbol schematics_library_legacy:root_0_Fiducial 1.3_schematics_library_legacy.schlib
- removed MEC1, MEC2, MEC3, MEC4, MEC5, MEC6, MEC7, MEC8, MEC9: M3, M3 hole, symbol schematics_library_legacy:root_0_M3 hole_schematics_library_legacy.schlib
- added C26: 0.01uF/50V, CC0805, symbol PCB_Project_FlightModel_EPS:dc_dc_3V3_OBDH_and_3V3_Deployment_ANT_1_Cap_Cer_X7R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
- added C27, C29: 0.1uF/50V, CC0805, symbol PCB_Project_FlightModel_EPS:dc_dc_3V3_OBDH_and_3V3_Deployment_ANT_0_Cap_Cer_X7R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
- added C28: 10uF/25V, CC1206, symbol PCB_Project_FlightModel_EPS:dc_dc_3V3_OBDH_and_3V3_Deployment_ANT_0_Cap_Cer_X7R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
- added C30: 22uF/10V, CC1206, symbol PCB_Project_FlightModel_EPS:dc_dc_3V3_OBDH_and_3V3_Deployment_ANT_0_Cap_Cer_X7R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
- added C31: 220uF/6.3V, FloripaSatPcbLib.PcbLib:cc1210, symbol PCB_Project_FlightModel_EPS:dc_dc_3V3_OBDH_and_3V3_Deployment_ANT_0_Cap_Tant_SM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
- added D4: B340LA-13-F, DO-214AC, symbol PCB_Project_FlightModel_EPS:dc_dc_3V3_OBDH_and_3V3_Deployment_ANT_1_DIODE_SCHOT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
- added J1, J2: 2053380002, footprints:2053380002, symbol 3V3_eps2_converter:2053380002
- added J3: 53261-0571, 532610571TR250, symbol 3V3_eps2_converter:53261-0571
- added L4: 16uH/5A/34.5mOHM, IND_744325xxx, symbol PCB_Project_FlightModel_EPS:dc_dc_3V3_OBDH_and_3V3_Deployment_ANT_1_IND_POWER_1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
- added R2, R4: 5m, footprints:RES2010, symbol 3V3_eps2_converter:WSL20105L000FEA
- added R20: 0R, 1206, symbol PCB_Project_FlightModel_EPS:dc_dc_3V3_OBDH_and_3V3_Deployment_ANT_1_R0R_JUMPER_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
- added R22: 10k, 0805, symbol PCB_Project_FlightModel_EPS:dc_dc_3V3_OBDH_and_3V3_Deployment_ANT_0_R10k_1%_1/8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
- added R24: 5K9, 0805, symbol PCB_Project_FlightModel_EPS:dc_dc_3V3_OBDH_and_3V3_Deployment_ANT_0_R5.9K_1%_1/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
- added U4: ${PARTNUMBER}, SO8 Power PAD, symbol PCB_Project_FlightModel_EPS:dc_dc_3V3_OBDH_and_3V3_Deployment_ANT_0_TPS5420QDRQ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
Connections:
- new net: J3.4, R20.2, R4.2
- new net: C27.1, C28.1, R20.1, U4.5 (ENA), U4.7 (VIN)
- new net: C29.1, C30.1, C31.1, J3.2, L4.2, R2.1, R22.2
- new net: J2.1, J3.1, R2.2
- new net: C26.1, U4.1 (BOOT)
- new net: R22.1, R24.2, U4.4 (VSENSE)
- new net: C26.2, D4.1 (K), L4.1, U4.8 (PH)
- new net PGND: C27.2, C28.2, C29.2, C30.2, C31.2, D4.2 (A), J1.2, J2.2, J3.3, R24.1, U4.6 (GND), U4.9 (POWER_PAD)
- new net VBus: J1.1, J3.5, R4.1
- no-connect marks 8 -> 0
Other:
- removed sheet Interface
- note removed: "${##}"
- note removed: "${#}"
- note removed: "${CURRENT_DATE}"
- note removed: "${DESIGNEDBY}"
- note removed: "${PROJECTCODE}"
- note removed: "${PROJECTNAME} / ${VARIANTNAME}"
- note removed: "${PROJECTREVISION}"
- note removed: "${TITLE}"
- note removed: "0.1"
- note removed: "0.2"
- note removed: "0.3"
- note removed: "02-May-2023"
- note removed: "16-Jun-2021"
- note removed: "28-Aug-2020"
- note removed: "A3"
- note removed: "Andre M. P. Mattos"
- note removed: "Author"
- note removed: "Date"
- note removed: "Date:"
- note removed: "Description"
- note removed: "EPS 2 MCU diagram"
- note removed: "EPS 2 power diagram"
- note removed: "Engineer:"
- note removed: "FIDUTIALS"
- note removed: "João C. E. Barcellos"
- note removed: "MECHANICAL HOLES"
- note removed: "PCB"
- note removed: "PCB Elements"
- note removed: "Project Code:"
- note removed: "Project Contributions"
- note removed: "Project Information"
- note removed: "Project:"
- note removed: "Rev"
- note removed: "Revision History"
- note removed: "Revision:"
- note removed: "Sheet"
- note removed: "Size:"
- note removed: "SpaceLab - Federal University of Santa Catarina"
- note removed: "Title:"
- note removed: "Yan C. de Azeredo"
- note removed: "of"
