File: 3V3_eps2_converter/3V3_eps2_converter.kicad_pcb (KiCad board)
At the start: 4 copper layers, 92.1 x 89.1 mm, 53 parts, among them U4 TPS5420QDRQ1

Commit message: update
Routing:
- net Net3V3ANT_1: track 78.6 -> 79.5 mm
Changed lines of the file:
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@@
+	)
+	(segment
+		(start 424.35 107.66949)
+		(end 425.385 106.63449)
+		(width 0.508)
+		(layer "In1.Cu")
+		(net 102)
 	)
 	(segment
@@
 	)
 	(segment
-		(start 425.615 121.38862)
-		(end 425.615 106.86449)
+		(start 424.35 121.3)
+		(end 424.35 107.66949)
 		(width 0.508)
 		(layer "In1.Cu")
@@
 	)
 	(segment
-		(start 425.385 106.63449)
-		(end 425.615 106.86449)
+		(start 424.97064 121.92064)
+		(end 424.35 121.3)
 		(width 0.508)
 		(layer "In1.Cu")
@@
 	(segment
 		(start 425.08297 121.92064)
-		(end 425.615 121.38862)
+		(end 424.97064 121.92064)
 		(width 0.508)
 		(layer "In1.Cu")
@@
 	)
 	(segment
-		(start 441.425 106.61449)
+		(start 441.32051 105.55)
 		(end 441.905 106.13449)
+		(width 0.508)
+		(layer "In2.Cu")
+		(net 102)
+	)
+	(segment
+		(start 426.41949 105.55)
+		(end 441.32051 105.55)
+		(width 0.508)
+		(layer "In2.Cu")
+		(net 102)
+	)
+	(segment
+		(start 425.355 106.61449)
+		(end 426.41949 105.55)
 		(width 0.508)
 		(layer "In2.Cu")
@@
 		(width 0.508)
 		(layer "In2.Cu")
-		(net 102)
-	)
-	(segment
-		(start 425.355 106.61449)
-		(end 441.425 106.61449)
-		(width 0.508)
-		(layer "In2.Cu")

Commit message: needs review
Parts:
- removed +X, +Y, +Z, -X, -Y, -Z: Header 4_PicoBlade, FloripaSatPcbLib:HDR4 PicoBlade
- removed ? (x3): , 
- removed the C26 at (165.0, 109.6)
- removed the C27 at (173.5, 113.9)
- removed the C28 at (175.2, 114.6)
- removed the C29 at (177.2, 87.0)
- removed the C30 at (177.2, 89.9)
- removed the C31 at (177.3, 92.4)
- removed the D4 at (173.0, 108.6)
- removed FD1, FD2, FD3, FD4, FD5, FD6: Fiducial 1.3, footprints_library_legacy:Fiducial 1.3mm
- removed the L4 at (169.9, 100.1)
- removed MEC1, MEC2, MEC3, MEC4, MEC5, MEC6, MEC7, MEC8, MEC9: M3, footprints_library_legacy:M3 hole
- removed PC104: PC104, FloripaSatPcbLib:PC104
- removed the R20 at (177.3, 114.7)
- removed the R22 at (160.7, 113.7)
- removed the R24 at (160.7, 109.7)
- removed RBF: 0533980471, footprints_library_legacy:PICOBLADE 4PIN VERTICAL
- removed R_ESD: 1.2M, PCB_EPS_2:0805
- removed SBW: 0532610671, footprints_library_legacy:PICOBLADE 6PIN Right Angle
- removed the U4 at (165.3, 111.5)
- removed UART: DNP, footprints_library_legacy:HDR 1X3
- moved C26 294.5 mm to (136.8, 99.8)
- moved C27 294.5 mm to (145.3, 104.0)
- moved C28 294.5 mm to (147.0, 104.7)
- moved C29 294.5 mm to (149.0, 77.1)
- moved C30 294.5 mm to (149.0, 80.1)
- moved C31 294.5 mm to (149.1, 82.6)
- moved D4 294.5 mm to (144.8, 98.8)
- moved L4 294.5 mm to (141.7, 90.2)
- moved R20 294.5 mm to (149.1, 104.8)
- moved R22 294.5 mm to (132.5, 103.8)
- moved R24 294.5 mm to (132.5, 99.9)
- moved U4 294.5 mm to (137.1, 101.6)
Routing:
- net VBus: track 343.8 -> 0.00 mm, vias 10 -> 0
- net 3V3_M: track 256.5 -> 0.00 mm, vias 19 -> 0
- net 3V3_MCU: track 213.4 -> 0.00 mm, vias 14 -> 0
- net 3V3_EPS_BEACON: track 152.7 -> 0.00 mm, vias 4 -> 0
- net UART_DEBUG_TX: track 106.7 -> 0.00 mm, vias 3 -> 0
- net UART_DEBUG_RX: track 98.7 -> 0.00 mm, vias 3 -> 0
- net En_5V_Radio_0: track 95.5 -> 0.00 mm, vias 2 -> 0
- net +RBF: track 93.9 -> 0.00 mm, vias 4 -> 0
- net NetC128_2: track 93.6 -> 0.00 mm, vias 3 -> 0
- net A3V3_EPS: track 91.7 -> 0.00 mm, vias 7 -> 0
- net I2C1_SCL_BUF: track 87.4 -> 0.00 mm, vias 4 -> 0
- net ADC1_V: track 87.1 -> 0.00 mm, vias 3 -> 0
- net En_6V_Radio_1: track 86.6 -> 0.00 mm, vias 2 -> 0
- net 5V_PAYLOAD: track 84.7 -> 0.00 mm
- net I2C1_SDA_BUF: track 84.6 -> 0.00 mm, vias 3 -> 0
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- removed copper zone on B.Cu, net +RBF
- removed copper zone on In1.Cu, net +RBF
- removed copper zone on B.Cu, net -VBAT
- removed copper zone on In1.Cu, net -VBAT
- removed copper zone on F.Cu, net 6V_Radio_1
- removed copper zone on B.Cu, net AGND
- removed copper zone on B.Cu, net DGND
- removed copper zone on In2.Cu, net DGND
- removed copper zone on F.Cu, net Net3V3OBDH_1
- removed copper zone on F.Cu, net NetC11_2
- removed copper zone on F.Cu, net NetC15_1
- removed copper zone on F.Cu, net NetC1_2
- removed copper zone on F.Cu, net NetC21_2
- removed copper zone on F.Cu, net NetC44_2
- removed copper zone on F.Cu, net NetC47_2
- removed copper zone on F.Cu, net NetC52_2
- removed copper zone on F.Cu, net NetC55_1
- removed copper zone on F.Cu, net NetC5_1
- removed copper zone on B.Cu, net PGND
- removed copper zone on In1.Cu, net PGND
- removed copper zone on In2.Cu, net PGND
- removed copper zone on F.Cu, net VPANELS
- removed copper zone on B.Cu, net V_CHARGING_BATTERIES
Other:
- board size 92.1 x 89.1 mm -> 29 x 39 mm
- board text removed: "${DESIGNATOR}"
- board text removed: "'.Layer_Name'"
- board text removed: "'.Print_Date'"
- board text removed: "+"
- board text removed: "-"
- board text removed: "0,010mm"
- board text removed: "0,035mm"
- board text removed: "0,036mm"
- board text removed: "0,110mm"
- board text removed: "0,300mm (11,81mil)"
- board text removed: "0,381mm (15,00mil)"
- board text removed: "0,600mm (23,62mil)"
- board text removed: "0,711mm (28,00mil)"
- board text removed: "0,900mm (35,43mil)"
- board text removed: "0,991mm (39,00mil)"
- board text removed: "1"
- board text removed: "1,000mm (39,37mil)"
- board text removed: "1,200mm"
- board text removed: "104"
- board text removed: "16"
- board text removed: "2"
- board text removed: "24"
- board text removed: "253"
- board text removed: "3"
- board text removed: "3,200mm (125,98mil)"
- board text removed: "3.5"
- board text removed: "32"
- board text removed: "4"
- board text removed: "4.2"
- board text removed: "40"
- board text removed: "44"
- board text removed: "46"
- board text removed: "5"
- board text removed: "502 Total"
- board text removed: "5V_OBDH"
- board text removed: "5V_PAYLOAD"
- board text removed: "5V_RADIO_0"
- board text removed: "6V_RADIO_1"
- board text removed: "77"
- board text removed: "8"
- board text removed: "9"
- board text removed: "A"
- board text removed: "A4"
- board text removed: "ADD_GPIO"
- board text removed: "ADD_I2C"
- board text removed: "AGND"
- board text removed: "ANT_VCC"
- board text removed: "Andre M. P. Mattos (based on FSat-I EPS)"
- board text removed: "Assembly specifications:"
- board text removed: "B"
- board text removed: "BATTERY"
- board text removed: "BAT_VCC"
- board text removed: "Board Layer Stack"
- board text removed: "Bottom Layer"
- board text removed: "Bottom Overlay"
- board text removed: "Bottom Solder"
- board text removed: "C"
- board text removed: "CHARGER"
- board text removed: "CK"
- board text removed: "Constant"
- board text removed: "Copper"
- board text removed: "Core"
- board text removed: "Count"
- board text removed: "D"
- board text removed: "DGND"
- board text removed: "DO"
- board text removed: "Date:"
- board text removed: "Designed by:"
- board text removed: "Dielectric 1"
- board text removed: "Dielectric 2"
- board text removed: "Drill Layer Pair"
- board text removed: "EN_RADIOS"
- board text removed: "EPS2"
- board text removed: "EPS_I2C"
- board text removed: "FR-4"
- board text removed: "Fabrication specifications:"
- board text removed: "GND"
- board text removed: "GPIO"
- board text removed: "H1+"
- board text removed: "H1-"
- board text removed: "H2-"
- board text removed: "HEATER"
- board text removed: "Hole Size"
- board text removed: "Hole Type"
- board text removed: "JTAG"
- board text removed: "Layer"
- board text removed: "Layer:"
- board text removed: "Material"
- board text removed: "NC1"
- board text removed: "NC2"
- board text removed: "Name"
- board text removed: "PGND"
- board text removed: "PTH"
- board text removed: "Pad"
- board text removed: "Plated"
- board text removed: "Project Code:"
- board text removed: "Project:"
- board text removed: "RBF+"
- board text removed: "RBF-"
- board text removed: "RTD"
- board text removed: "RTD0"
- board text removed: "RTD1"
- board text removed: "RTD2"
- board text removed: "RTD3"
- board text removed: "RTD4"
- board text removed: "RTD5"
- board text removed: "RTD6"
- board text removed: "RX"
- board text removed: "Round"
- board text removed: "Signal Layer 1"
- board text removed: "Signal Layer 2"
- board text removed: "Size:"
- board text removed: "Solder Resist"
- board text removed: "SpaceLab - Federal University of Santa Catarina"
- board text removed: "Symbol"
- board text removed: "TP1"
- board text removed: "TP2"
- board text removed: "TP9"
- board text removed: "TX"
- board text removed: "Thickness"
- board text removed: "Top Layer"
- board text removed: "Top Layer - Bottom Layer"
- board text removed: "Top Overlay"
- board text removed: "Top Solder"
- board text removed: "UART_RADIO_1"
- board text removed: "V+"
- board text removed: "V-"
- board text removed: "VBAT+"
- board text removed: "VBAT-"
- board text removed: "VBus_TP"
- board text removed: "VCC"
- board text removed: "V_CM"
- board text removed: "Version:"
- board text removed: "Via"
- board text removed: "Via/Pad"
- board text removed: "v0.3"
